File: hardware/outputs/NIVA-3D-engineering-prototype/electronics/NIVA-pod.kicad_pcb (KiCad board)
At the start: 4 copper layers, 34 x 48 mm, 66 parts, among them J1 INSERT TAIL (JST GH 10, keyed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, J2 CARTRIDGE SPRING CONTACTS (pa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, J3 SERVICE PADS (TC2030-NL, unde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, SW1 KMR221G (C&K KMR2), U1 ESP32-C3-MINI-1-N4, U2 MCP3208-CI/SL, U3 LSM6DSO32TR, U4 MCP6001T-I/OT, U5 TLV75533PDBVR, U6 MAX17048G+T10

Commit message: NIVA Rev C: documentation, final exports, captioned PCB renders
- ELECTRICAL-REVIEW.md, PRINT-AND-ASSEMBLY.md and package README
- R33 raised to 220R (22R would dissipate 0.5 W in an 0603 on a tail short)
- deterministic schematic UUIDs; generators accept only KiCad 9 libraries
- regenerated ERC/netlist/BOM/PCB/DRC/PCBA STEP+GLB/assembly PDFs
- Blender scene builder and caption tool; KiCad raytraced PCB views
- stale Rev B generated outputs removed (kept in git history)

Co-Authored-By: Claude Opus 5.5 <noreply@anthropic.com>
Claude-Session: https://claude.ai/code/session_01HNzeJFE5uNHjapog53SHnm
Parts:
- R33: value 22 -> 220

Commit message: Add cartridge interconnect PCB, charging dock PCB and dock enclosure; ratiometric ADC reference
- Pod schematic: MCP3208 VREF driven from VEXC (the sensor excitation rail) so every
  channel is ratiometric in hardware; CH6 reads +3V3/2 as a rail monitor.
- Cartridge: 3.4 mm interconnect strip (cell leads, polyfuse, lid-plate leads, underside
  dock pads), hand-routed; ERC/DRC clean with schematic parity.
- Dock: USB-C sink, MCP73831 charger gated by an LM393 NTC window comparator, spring
  pins to the cartridge pads; autorouted (Freerouting) and DRC clean.
- Fabrication data for both boards written only as review-only sets with open blockers.
- Dock enclosure (base, top with keyed well, tab ledge, snap latch, light pipe) generated
  from niva_layout.py; interference audit reports only the expected spring-pin contacts.
- Shared CAD helpers and cartridge builders moved to niva_cad_lib.py.

Co-Authored-By: Claude Opus 5.5 <noreply@anthropic.com>
Claude-Session: https://claude.ai/code/session_01HNzeJFE5uNHjapog53SHnm
Parts:
- R31, R32: value 10k 0.1% -> 10k 1%
- moved C4 9.10 mm to (107.0, 68.4), turned to 0 degrees
- moved C8 8.22 mm to (131.0, 61.8), turned to 0 degrees
- moved R45 7.00 mm to (126.4, 67.6)
- moved R46 4.12 mm to (126.4, 69.4)
- moved C19 3.94 mm to (111.0, 68.4), turned to 0 degrees
- moved U2 3.94 mm to (111.0, 74.0), turned to 90 degrees
- moved D4 3.70 mm to (119.4, 68.5)
- moved D5 3.70 mm to (122.8, 68.5)
Connections:
- net /Controller/VEXC_HALF renamed /Controller/V33_HALF
- C19 pad 1: +3V3 -> /Controller/VEXC
- R30 pad 1: +3V3 -> /Controller/VEXC
- R31 pad 1: /Controller/VEXC -> +3V3
- R40 pad 1: +3V3 -> /Controller/VEXC
- U2 pad 15: +3V3 -> /Controller/VEXC
Other:
- board text removed: "ENGINEERING PROTOTYPE - NOT FOR FABRICATION"
- board text removed: "UNROUTED PLACEMENT PROTOTYPE - RATSNEST ONLY - NOT FOR FABRICATION"

Commit message: Route the pod PCB, add BAV199 clamp, insole sensing flex, verification plan
- Pod: 0.15/0.127 mm rules; every GND pad fanned out to the In1 plane before
  autorouting, signals routed with Freerouting, GND pours stitched on all layers.
  KiCad DRC: 0 errors, 0 unconnected, schematic parity clean.
- D2/D3 BAS416 singles replaced by one BAV199 series pair on a project symbol
  that states the datasheet pinning.
- Insole flex (right/left medium): five interdigitated shunt-mode electrodes,
  PVDF bond pads, paired lanes to the heel tab, above-collar transition with the
  insert ID resistor; F.Cu only and no parts underfoot. ERC/DRC clean.
- export_niva_electronics.py writes all board outputs; fabrication data only in
  per-board fab-REVIEW-ONLY-NOT-RELEASED folders with open blockers.
- VERIFICATION-PLAN.md: sealing, skin-contact and cleaning test plan (no claims).
- Dock CAD re-audited against the new dock STEP; pod CAD against the routed PCBA.
- Blender import linearises KiCad GLB colours; dock and insole-flex scenes added.
- README, ELECTRICAL-REVIEW and PRINT-AND-ASSEMBLY updated for Rev C.1.

Co-Authored-By: Claude Opus 5.5 <noreply@anthropic.com>
Claude-Session: https://claude.ai/code/session_01HNzeJFE5uNHjapog53SHnm
Parts:
- removed D3: BAS416, Diode_SMD:D_SOD-323
- D2: value BAS416 -> BAV199; footprint Diode_SMD:D_SOD-323 -> Package_TO_SOT_SMD:SOT-23
- moved D2 0.65 mm to (131.5, 82.1)
Connections:
- D2 pad 1: +3V3 -> GND
- D2 pad 2: /Heel and indicator/PZ_BIAS -> +3V3
Routing:
- net +3V3: track 0.00 -> 130.3 mm, vias 0 -> 1
- net GND: track 0.00 -> 69.8 mm, vias 0 -> 81
- net /Controller/VEXC: track 0.00 -> 49.6 mm, vias 0 -> 4
- net VBAT: track 0.00 -> 43.6 mm, vias 0 -> 1
- net /Controller/CHIP_EN: track 0.00 -> 39.9 mm, vias 0 -> 2
- net /Controller/SPI_SCK: track 0.00 -> 38.6 mm, vias 0 -> 2
- net /Controller/BOOT9: track 0.00 -> 35.2 mm, vias 0 -> 2
- net /Controller/BUTTON: track 0.00 -> 34.9 mm, vias 0 -> 3
- net /Controller/I2C_SCL: track 0.00 -> 31.2 mm, vias 0 -> 2
- net /Controller/I2C_SDA: track 0.00 -> 30.7 mm, vias 0 -> 2
- net /Controller/SPI_MISO: track 0.00 -> 30.4 mm, vias 0 -> 2
- net /Controller/SPI_MOSI: track 0.00 -> 28.0 mm, vias 0 -> 2
- net /Controller/INSERT_ID: track 0.00 -> 26.7 mm, vias 0 -> 2
- net /Controller/V33_HALF: track 0.00 -> 21.5 mm, vias 0 -> 2
- net /Controller/CS_IMU: track 0.00 -> 21.4 mm, vias 0 -> 2
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- added copper zone on B.Cu, net GND
- added copper zone on F.Cu, net GND
- added copper zone on In2.Cu, net GND
Other:
- board text added: "ROUTED PROTOTYPE - SIGNALS FREEROUTING, GND FAN-OUT + POURS - DRC CHECKED - NOT RELEASED"
