File: hardware/outputs/NIVA-3D-engineering-prototype/electronics/NIVA-pod.kicad_pcb (KiCad board)
At the start: 4 copper layers, 34 x 48 mm, 65 parts, among them J1 INSERT TAIL (JST GH 10, keyed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, J2 CARTRIDGE SPRING CONTACTS (pa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, J3 SERVICE PADS (TC2030-NL, unde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, SW1 KMR221G (C&K KMR2), U1 ESP32-C3-MINI-1-N4, U2 MCP3208-CI/SL, U3 LSM6DSO32TR, U4 MCP6001T-I/OT, U5 TLV75533PDBVR, U6 MAX17048G+T10

Commit message: Pod PCB: add PCBWay text to bottom silkscreen
PCBWay's Future Innovators Program requires the PCBWay name or logo
on every supported board. Add "PCBWay" (1 mm, 0.15 mm stroke) on
B.Silkscreen under "NIVA REV C", in a spot clear of pads, vias and
other silk. Re-export the PCBWay Gerbers and zip; only the bottom
silkscreen changes (copper and drill differ by timestamp only).

KiCad 10.0.7 DRC with parity: 0 errors, 0 unconnected, same 13
warnings as before.

Co-Authored-By: Claude Opus 5.5 <noreply@anthropic.com>
Other:
- board text added: "PCBWay"
Changed lines of the file:
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@@
+		)
+	)
+	(gr_text "PCBWay"
+		(at 121 62.5 0)
+		(layer "B.SilkS")
+		(effects
+			(font
+				(size 1 1)
+				(thickness 0.15)
+			)
+			(justify mirror)
 		)
 	)
